Commit message: urdf changes

File: install/robot_description/share/robot_description/urdf/mycobot_with_vision_v2.urdf (robot description, URDF)
Before this commit: robot mycobot_ai, 8 links, 7 joints
Links:
- added link suction_pump; collision mesh filename=package://robot_description/urdf/SuctionPump.STL; visual mesh filename=package://robot_description/urdf/SuctionPump.STL
Joints:
- added joint joint6output_to_suction_pump: type fixed, parent joint6_flange, child suction_pump, origin xyz=0 0.30 0.30 rpy=0 0 0, axis 0 0 0, limit lower=-3.14 upper=3.14159 effort=1000.0 velocity=0

Commit message: changed urdf

File: install/robot_description/share/robot_description/urdf/mycobot_with_vision_v2.urdf (robot description, URDF)
Before this commit: robot mycobot_ai, 9 links, 8 joints
Links:
- link suction_pump: geometry collision mesh filename=package://robot_description/urdf/SuctionPumpInches.STL; visual mesh filename=package://robot_description/urdf/SuctionPumpInches.STL
Joints:
- joint joint6output_to_suction_pump: origin xyz=0 0.30 0.30 rpy=0 0 0 -> xyz=0 0.030 0.030 rpy=0 0 0

Commit message: moveit_config

File: install/robot_description/share/robot_description/urdf/mycobot_with_vision_v2.urdf (robot description, URDF)
Before this commit: robot mycobot_ai, 9 links, 8 joints
Links:
- link suction_pump: geometry collision mesh filename=package://robot_description/urdf/SuctionPumpMeters.STL; visual mesh filename=package://robot_description/urdf/SuctionPumpMeters.STL
Joints:
- joint joint6output_to_suction_pump: origin xyz=0 0.030 0.030 rpy=0 0 0 -> xyz=0 0 0 rpy=0 0 0

Commit message: changes

File: install/robot_description/share/robot_description/urdf/mycobot_with_vision_v2.urdf (robot description, URDF)
Before this commit: robot mycobot_ai, 9 links, 8 joints
Links:
- link env: geometry collision mesh filename=package://robot_description/urdf/env_meters.STL; visual mesh filename=package://robot_description/urdf/suit_env_v2.dae

Commit message: Robot moves!

File: install/robot_description/share/robot_description/urdf/mycobot_with_vision_v2.urdf (robot description, URDF)
Before this commit: robot mycobot_ai, 9 links, 8 joints
Links:
- link env: geometry collision mesh filename=package://robot_description/urdf/env_meters_correct_coords.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; visual mesh filename=package://robot_description/urdf/suit_env_v2.dae
