Commit message: lots of stuff

File: install/moveit_config/share/moveit_config/config/mycobot_ai.ros2_control.xacro (robot description, xacro)
@@ -1,48 +1 @@
-<?xml version="1.0"?>
-<robot xmlns:xacro="http://www.ros.org/wiki/xacro">
-    <xacro:macro name="mycobot_ai_ros2_control" params="name initial_positions_file">
-        <xacro:property name="initial_positions" value="${load_yaml(initial_positions_file)['initial_positions']}"/>
-        <ros2_control name="${name}" type="system">
-            <hardware>
-                <!-- By default, set up controllers for simulation. This won't work on real hardware -->
-                <plugin>mock_components/GenericSystem</plugin>
-            </hardware>
-            <joint name="joint2_to_joint1">
-                <command_interface name="position"/>
-                <state_interface name="position">
-                  <param name="initial_value">${initial_positions['joint2_to_joint1']}</param>
-                </state_interface>
-            </joint>
-            <joint name="joint3_to_joint2">
-                <command_interface name="position"/>
-                <state_interface name="position">
-                  <param name="initial_value">${initial_positions['joint3_to_joint2']}</param>
-                </state_interface>
-            </joint>
-            <joint name="joint4_to_joint3">
-                <command_interface name="position"/>
-                <state_interface name="position">
-                  <param name="initial_value">${initial_positions['joint4_to_joint3']}</param>
-                </state_interface>
-            </joint>
-            <joint name="joint5_to_joint4">
-                <command_interface name="position"/>
-                <state_interface name="position">
-                  <param name="initial_value">${initial_positions['joint5_to_joint4']}</param>
-                </state_interface>
-            </joint>
-            <joint name="joint6_to_joint5">
-                <command_interface name="position"/>
-                <state_interface name="position">
-                  <param name="initial_value">${initial_positions['joint6_to_joint5']}</param>
-                </state_interface>
-            </joint>
-            <joint name="joint6output_to_joint6">
-                <command_interface name="position"/>
-                <state_interface name="position">
-                  <param name="initial_value">${initial_positions['joint6output_to_joint6']}</param>
-                </state_interface>
-            </joint>
-        </ros2_control>
-    </xacro:macro>
-</robot>
+/home/lance/robot/src/moveit_config/config/mycobot_ai.ros2_control.xacro

File: install/moveit_config/share/moveit_config/config/mycobot_ai.urdf.xacro (robot description, xacro)
@@ -1,9 +1 @@
-<?xml version="1.0"?>
-<robot xmlns:xacro="http://www.ros.org/wiki/xacro" name="mycobot_ai">
-    <xacro:arg name="initial_positions_file" default="initial_positions.yaml" />
-    <!-- Import mycobot_ai urdf file -->
-    <xacro:include filename="$(find robot_description)/urdf/mycobot_with_vision_v2.urdf" />
-    <!-- Import control_xacro -->
-    <xacro:include filename="mycobot_ai.ros2_control.xacro" />
-    <xacro:mycobot_ai_ros2_control name="FakeSystem" initial_positions_file="$(arg initial_positions_file)"/>
-</robot>
+/home/lance/robot/src/moveit_config/config/mycobot_ai.urdf.xacro

File: src/moveit_config/config/mycobot_ai.ros2_control.xacro (robot description, xacro)
@@ -6,5 +6,5 @@
             <hardware>
                 <!-- By default, set up controllers for simulation. This won't work on real hardware -->
-                <plugin>mock_components/GenericSystem</plugin>
+                <plugin>my_cobot_hardware_interface</plugin>
             </hardware>
             <joint name="joint2_to_joint1">

Commit message: IK added and functional, camera and robot coordinate systems aligned

File: install/moveit_config/share/moveit_config/config/mycobot_ai.ros2_control.xacro (robot description, xacro)
@@ -1 +1,47 @@
-/home/lance/robot/src/moveit_config/config/mycobot_ai.ros2_control.xacro
+<?xml version="1.0"?>
+<robot xmlns:xacro="http://www.ros.org/wiki/xacro">
+    <xacro:macro name="mycobot_ai_ros2_control" params="name initial_positions_file">
+        <xacro:property name="initial_positions" value="${load_yaml(initial_positions_file)['initial_positions']}"/>
+        <ros2_control name="${name}" type="actuator">
+            <hardware>
+                <!-- <plugin>my_cobot_hardware_interface/MyCobotHardwareInterface</plugin> -->
+            </hardware>
+            <joint name="joint2_to_joint1">
+                <command_interface name="position"/>
+                <state_interface name="position">
+                  <param name="initial_value">${initial_positions['joint2_to_joint1']}</param>
+                </state_interface>
+            </joint>
+            <joint name="joint3_to_joint2">
+                <command_interface name="position"/>
+                <state_interface name="position">
+                  <param name="initial_value">${initial_positions['joint3_to_joint2']}</param>
+                </state_interface>
+            </joint>
+            <joint name="joint4_to_joint3">
+                <command_interface name="position"/>
+                <state_interface name="position">
+                  <param name="initial_value">${initial_positions['joint4_to_joint3']}</param>
+                </state_interface>
+            </joint>
+            <joint name="joint5_to_joint4">
+                <command_interface name="position"/>
+                <state_interface name="position">
+                  <param name="initial_value">${initial_positions['joint5_to_joint4']}</param>
+                </state_interface>
+            </joint>
+            <joint name="joint6_to_joint5">
+                <command_interface name="position"/>
+                <state_interface name="position">
+                  <param name="initial_value">${initial_positions['joint6_to_joint5']}</param>
+                </state_interface>
+            </joint>
+            <joint name="joint6output_to_joint6">
+                <command_interface name="position"/>
+                <state_interface name="position">
+                  <param name="initial_value">${initial_positions['joint6output_to_joint6']}</param>
+                </state_interface>
+            </joint>
+        </ros2_control>
+    </xacro:macro>
+</robot>

File: install/moveit_config/share/moveit_config/config/mycobot_ai.urdf.xacro (robot description, xacro)
@@ -1 +1,9 @@
-/home/lance/robot/src/moveit_config/config/mycobot_ai.urdf.xacro
+<?xml version="1.0"?>
+<robot xmlns:xacro="http://www.ros.org/wiki/xacro" name="mycobot_ai">
+    <xacro:arg name="initial_positions_file" default="initial_positions.yaml" />
+    <!-- Import mycobot_ai urdf file -->
+    <xacro:include filename="$(find robot_description)/urdf/mycobot_with_vision_v2.urdf" />
+    <!-- Import control_xacro -->
+    <xacro:include filename="mycobot_ai.ros2_control.xacro" />
+    <xacro:mycobot_ai_ros2_control name="FakeSystem" initial_positions_file="$(arg initial_positions_file)"/>
+</robot>

File: src/moveit_config/config/mycobot_ai.ros2_control.xacro (robot description, xacro)
@@ -3,8 +3,7 @@
     <xacro:macro name="mycobot_ai_ros2_control" params="name initial_positions_file">
         <xacro:property name="initial_positions" value="${load_yaml(initial_positions_file)['initial_positions']}"/>
-        <ros2_control name="${name}" type="system">
+        <ros2_control name="${name}" type="actuator">
             <hardware>
-                <!-- By default, set up controllers for simulation. This won't work on real hardware -->
-                <plugin>my_cobot_hardware_interface</plugin>
+                <!-- <plugin>my_cobot_hardware_interface/MyCobotHardwareInterface</plugin> -->
             </hardware>
             <joint name="joint2_to_joint1">
